File: matrix-clock-pcb/matrix-clock.sch (KiCad schematic (older format))
At the start: 15 parts

Commit message: pcb: update pcb files
Parts:
- added C5, C6: 0.1uf, Capacitor_SMD:C_0402_1005Metric, symbol Device:C
- J2: renamed from J?; symbol Connector_Generic:Conn_02x08_Counter_Clockwise -> Connector_Generic:Conn_02x08_Odd_Even
- gave numbers to parts that had none: 14
Connections:
- net labels added: _LED_A, _LED_B, _LED_C, _LED_D, _LED_G1, _LED_G2, _LED_OE, _LED_R1, _LED_R2, _LED_SCK, _LED_STCP
- wire segments 79 -> 80
Other:
- moved on the sheet: U3, U4

Commit message: pcb: update pcb to v1.1
Parts:
- removed U3, U4: TXB0108PWR, Package_SO:TSSOP-20_4.4x6.5mm_P0.65mm, symbol mylib:TXB0108PWR
- added U3, U4: 74HC245, Package_SO:TSSOP-20_4.4x6.5mm_P0.65mm, symbol 74xx:74HC245
Connections:
- net +3V3: no longer C5.2
- net +5V: now also C5.2, U3.1 (A->B), U3.20 (VCC), U4.1 (A->B), U4.20 (VCC)
- net GND: now also U3.10 (GND), U3.19 (CE), U4.10 (GND), U4.19 (CE)
- net LED_A: now also U3.9 (A7)
- net LED_B: now also U3.8 (A6)
- net LED_C: now also U3.7 (A5)
- net LED_D: now also U3.6 (A4)
- net LED_G1: now also U3.5 (A3)
- net LED_G2: now also U3.4 (A2)
- net LED_OE: now also U4.4 (A2)
- net LED_R1: now also U4.3 (A1)
- net LED_R2: now also U4.2 (A0)
- net LED_SCK: now also U3.2 (A0)
- net LED_STCP: now also U3.3 (A1)
- net _LED_A: now also U3.11 (B7)
- net _LED_B: now also U3.12 (B6)
- net _LED_C: now also U3.13 (B5)
- net _LED_D: now also U3.14 (B4)
- net _LED_G1: now also U3.15 (B3)
- net _LED_G2: now also U3.16 (B2)
- net _LED_OE: now also U4.16 (B2)
- net _LED_R1: now also U4.17 (B1)
- net _LED_R2: now also U4.18 (B0)
- net _LED_SCK: now also U3.18 (B0)
- net _LED_STCP: now also U3.17 (B1)
Other:
- moved on the sheet: C5, C6, J2

Commit message: fix(pcb): modify cp2102 IO voltage to 3.3v; add ir receiver
Parts:
- added C?: 0.1uf, Capacitor_SMD:C_0402_1005Metric, symbol Device:C
- added J?: Conn_01x03, symbol Connector_Generic:Conn_01x03
- added R?: 10K, Resistor_SMD:R_0402_1005Metric, symbol Device:R
Connections:
- net +3V3: now also C?.1, J?.3 (Pin_3), R?.1
- net GND: now also C?.2, J?.2 (Pin_2)
- net IR_SIGNAL: now reaches U1.9 (IO33)
- net IR_SIGNAL: now also J?.1 (Pin_1), R?.2
- no-connect marks 23 -> 22
Changed lines of the file:
@@
 	1    0    0    -1
 $EndComp
-Text Label 2450 6150 0    50   ~ 0
-RXD0
-Text Label 2450 6350 0    50   ~ 0
-BOOT
-Text Label 2450 6250 0    50   ~ 0
-EN
-Text Label 2450 6050 0    50   ~ 0
-TXD0
-Wire Wire Line
-	2300 6050 2450 6050
-Wire Wire Line
-	2300 6150 2450 6150
-Wire Wire Line
-	2300 6250 2450 6250
-Wire Wire Line
-	2300 6350 2450 6350
-$Sheet
-S 1050 5900 1250 650
-U 5F4ECFED
-F0 "Sheet5F4ECFED" 50
-F1 "power.sch" 50
-F2 "CHIP_IO0" O R 2300 6350 50
-F3 "CHIP_EN" O R 2300 6250 50
-F4 "TXD" O R 2300 6150 50
-F5 "RXD" I R 2300 6050 50
-$EndSheet
 $Comp
 L Connector_Generic:Conn_02x08_Odd_Even J2
@@
 $EndComp
 Connection ~ 5600 2100
-NoConn ~ 3450 3950
 NoConn ~ 3450 4050
 NoConn ~ 3450 4150
@@
 	0    1    1    0
 $EndComp
+$Comp
+L Connector_Generic:Conn_01x03 J?
+U 1 1 604711F6
+P 1150 5200
+F 0 "J?" H 1250 4850 50  0000 C CNN
+F 1 "Conn_01x03" H 1200 4950 50  0000 C CNN
+F 2 "" H 1150 5200 50  0001 C CNN
+F 3 "~" H 1150 5200 50  0001 C CNN
+	1    1150 5200
+	-1   0    0    1
+$EndComp
+$Comp
+L power:GND #PWR?
+U 1 1 60472B23
+P 1550 5200
+F 0 "#PWR?" H 1550 4950 50  0001 C CNN
+F 1 "GND" H 1555 5027 50  0000 C CNN
+F 2 "" H 1550 5200 50  0001 C CNN
+F 3 "" H 1550 5200 50  0001 C CNN
+	1    1550 5200
+	0    -1   -1   0
+$EndComp
+$Comp
+L power:+3.3V #PWR?
+U 1 1 60474054
+P 1500 4900
+F 0 "#PWR?" H 1500 4750 50  0001 C CNN
+F 1 "+3.3V" H 1515 5073 50  0000 C CNN
+F 2 "" H 1500 4900 50  0001 C CNN
+F 3 "" H 1500 4900 50  0001 C CNN
+	1    1500 4900
+	1    0    0    -1
+$EndComp
+$Comp
+L Device:C C?
+U 1 1 60476314
+P 1500 5050
+F 0 "C?" H 1600 5050 50  0000 L CNN
+F 1 "0.1uf" H 1500 4950 50  0000 L CNN
+F 2 "Capacitor_SMD:C_0402_1005Metric" H 1538 4900 50  0001 C CNN
+F 3 "~" H 1500 5050 50  0001 C CNN
+	1    1500 5050
+	1    0    0    -1
+$EndComp
+Wire Wire Line
+	1550 5200 1500 5200
+Connection ~ 1500 5200
+Wire Wire Line
+	1500 5200 1350 5200
+Wire Wire Line
+	1350 5100 1350 4900
+Wire Wire Line
+	1350 4900 1500 4900
+Connection ~ 1500 4900
+Text Label 1950 5300 0    50   ~ 0
+IR_SIGNAL
+Text Label 3550 3950 0    50   ~ 0
+IR_SIGNAL
+Wire Wire Line
+	3450 3950 3550 3950
+$Comp
+L Device:R R?
+U 1 1 60480409
+P 1900 5050
+F 0 "R?" H 1970 5096 50  0000 L CNN
+F 1 "10K" H 1970 5005 50  0000 L CNN
+F 2 "Resistor_SMD:R_0402_1005Metric" V 1830 5050 50  0001 C CNN
+F 3 "~" H 1900 5050 50  0001 C CNN
+	1    1900 5050
+	1    0    0    -1
+$EndComp
+Wire Wire Line
+	1350 5300 1900 5300
+Wire Wire Line
+	1900 5200 1900 5300
+Connection ~ 1900 5300
+Wire Wire Line
+	1900 5300 1950 5300
+$Sheet
+S 1050 5900 1250 650
+U 5F4ECFED
+F0 "Sheet5F4ECFED" 50
+F1 "power.sch" 50
+F2 "CHIP_IO0" O R 2300 6350 50
+F3 "CHIP_EN" O R 2300 6250 50
+F4 "TXD" O R 2300 6150 50
+F5 "RXD" I R 2300 6050 50
+$EndSheet
+Wire Wire Line
+	2300 6350 2450 6350
+Wire Wire Line
+	2300 6250 2450 6250
+Wire Wire Line
+	2300 6150 2450 6150
+Wire Wire Line
+	2300 6050 2450 6050
+Text Label 2450 6050 0    50   ~ 0
+TXD0
+Text Label 2450 6250 0    50   ~ 0
+EN
+Text Label 2450 6350 0    50   ~ 0
+BOOT
+Text Label 2450 6150 0    50   ~ 0
+RXD0
+Wire Wire Line
+	1900 4900 1500 4900
 $EndSCHEMATC

Commit message: fix(pcb): update pcb layout
Parts:
- removed J?: Conn_01x03, symbol Connector_Generic:Conn_01x03
- added U8: VS1838, esp32:Infrared_Receiver_module, symbol mylib:VS1838
- gave numbers to parts that had none: 2
Connections:
- net +3V3: now also C15.2, R14.2, U8.3 (VCC); no longer C15.1, R14.1
- net GND: now also C15.1, U8.2 (GND); no longer C15.2
- net IR_SIGNAL: now also R14.1, U8.1 (OUT); no longer R14.2
- net SCL: now reaches R3.2, U1.26 (IO4), U2.2 (SCL)
- net SDA: now reaches R4.2, U1.29 (IO5), U2.3 (SDA)
Other:
- moved on the sheet: C15, C4, R14, R3, R4, U2
